File: electronics/lcd-unit-STM32/rayman_LCD_STM.kicad_pcb (KiCad board)
At the start: 4 copper layers, 70 x 80 mm, 92 parts, among them J1 Conn_01x02_Pin, J2 Conn_01x04_Pin, J3 Micro_SD_Card, J4 Conn_01x40, J5 Conn_01x04_Pin, SW2 SW_Push, U1 IS42S16400J-xT, U3 1808 SMD FUSEHOLDER, U4 MCP1826S-3302E/DB, U5 STM32H743IITx

Commit message: uv control fixed
Parts:
- removed D7: PUSB3TB6, moja:pus
- added U2: SP3012-06UTG, moja:SON50P350X135X55-14N, F.Cu at (126.4, 68.0)
Routing:
- net GND: track 91.8 -> 99.1 mm
- net pc11: track 34.9 -> 40.6 mm
- net Net-(J3-CMD): track 22.9 -> 19.9 mm, vias 1 -> 2
- net Net-(J3-CLK): track 12.0 -> 15.1 mm
- net pa12: track 95.5 -> 97.8 mm
- net pc9: track 80.2 -> 82.5 mm, vias 1 -> 3
- net nrst: track 100.4 -> 98.8 mm
- net swdio: track 33.6 -> 32.4 mm
- net pc8: track 80.0 -> 81.2 mm
- added copper zone on B.Cu, net GND

Commit message: Ambiente lighting draft, song order fixet for music rounds, many others
Parts:
- added C45: 4U7, Capacitor_SMD:C_0603_1608Metric, B.Cu at (113.2, 114.2)
- added C46: 100n, Capacitor_SMD:C_0603_1608Metric, B.Cu at (111.7, 114.1)
- added C47: 2.2u 50v, Capacitor_SMD:C_0603_1608Metric, B.Cu at (119.5, 124.9)
- added C48: 1uF, Capacitor_SMD:C_0603_1608Metric, B.Cu at (164.0, 97.9)
- added C49: 100nF, Capacitor_SMD:C_0603_1608Metric, B.Cu at (164.0, 96.4)
- added C50: 1uF, Capacitor_SMD:C_0603_1608Metric, B.Cu at (162.2, 105.0)
- added C51: 100nF, Capacitor_SMD:C_0603_1608Metric, B.Cu at (162.2, 103.4)
- added D7: D_Schottky, Diode_SMD:D_SMA, B.Cu at (115.8, 127.7)
- added L1: L, Inductor_SMD:L_Bourns-SRN4018, B.Cu at (107.0, 119.6)
- added R11: 10R, Resistor_SMD:R_0805_2012Metric, B.Cu at (116.1, 122.1)
- added R16: 100R, Resistor_SMD:R_0805_2012Metric, B.Cu at (112.1, 120.9)
- added R17: 100K, Resistor_SMD:R_0805_2012Metric, B.Cu at (112.1, 123.0)
- added R18: 4K7, Resistor_SMD:R_0805_2012Metric, B.Cu at (170.6, 88.4)
- added R19: 4K7, Resistor_SMD:R_0805_2012Metric, B.Cu at (168.1, 88.4)
- added R20: 4K7, Resistor_SMD:R_0805_2012Metric, B.Cu at (170.6, 106.7)
- added R21: 4K7, Resistor_SMD:R_0805_2012Metric, B.Cu at (168.1, 106.7)
- added U6: TPS61169DCKR, moja:SOT65P210X110-5N, B.Cu at (112.6, 117.8)
- moved R7 1.01 mm to (162.0, 124.0)
- moved J5 0.30 mm to (163.2, 101.3)
- moved J2 0.30 mm to (163.2, 93.5)
Connections:
- J2 pad 3: unconnected-(J2-SCK-Pad3) -> pb6
- J2 pad 4: unconnected-(J2-SDK-Pad4) -> pb7
- J4 pad 1: unconnected-(J4-ledk-Pad1) -> Net-(J4-ledk)
- J4 pad 2: unconnected-(J4-led_a-Pad2) -> Net-(D7-K)
- J5 pad 3: unconnected-(J5-SCK-Pad3) -> pb10
- J5 pad 4: unconnected-(J5-SDK-Pad4) -> ph5
- U5 pad 164: unconnected-(U5-PB6-Pad164) -> pb6
- U5 pad 165: unconnected-(U5-PB7-Pad165) -> pb7
- U5 pad 46: unconnected-(U5-PH5-Pad46) -> ph5
- U5 pad 53: unconnected-(U5-PA7-Pad53) -> gpio_stm32
- U5 pad 79: unconnected-(U5-PB10-Pad79) -> pb10
Routing:
- net ph5: track 0.00 -> 54.5 mm, vias 0 -> 2
- net pb7: track 0.00 -> 53.4 mm, vias 0 -> 2
- net pb6: track 0.00 -> 52.9 mm, vias 0 -> 2
- net +3V3: track 203.6 -> 246.3 mm, vias 26 -> 27
- net gpio_stm32: track 0.00 -> 40.9 mm, vias 0 -> 1
- net pb10: track 0.00 -> 33.0 mm
- net Net-(D7-A): track 0.00 -> 25.4 mm
- net Net-(D7-K): track 0.00 -> 22.4 mm, vias 0 -> 1
- net +5V: track 24.5 -> 35.7 mm
- net Net-(J4-ledk): track 0.00 -> 11.1 mm, vias 0 -> 1
- net Net-(U6-CTRL): track 0.00 -> 8.38 mm
- net pb0: track 40.0 -> 45.3 mm
- net pa8: track 75.6 -> 78.0 mm
- net pa10: track 79.0 -> 81.4 mm
- net GND: track 99.1 -> 101.3 mm, vias 30 -> 31
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Other:
- board text removed: "CAN_T"
