File: electronics/lcd-unit-STM32/rayman_LCD_STM.kicad_sch (KiCad schematic)
At the start: 31 parts, among them J1 Conn_01x02_Pin, J2 Conn_01x04_Pin, J5 Conn_01x04_Pin, SW2 SW_Push, U5 STM32H743IITx

Commit message: Ambiente lighting draft, song order fixet for music rounds, many others
Parts:
- added C48, C50: 1uF, Capacitor_SMD:C_0603_1608Metric, symbol Device:C_Small
- added C49, C51: 100nF, Capacitor_SMD:C_0603_1608Metric, symbol Device:C_Small
- added R18, R19, R20, R21: 4K7, Resistor_SMD:R_0805_2012Metric, symbol Device:R_Small
Connections:
- net +3V3: now also C48.1, C50.1, R18.2, R19.2, R20.2, R21.2
- net GND: now also C48.2, C50.2
- net pb6: now reaches U5.164 (PB6)
- net pb6: now also J2.3 (SCK), R19.1
- net pb7: now reaches U5.165 (PB7)
- net pb7: now also J2.4 (SDK), R18.1
- net ph5: now reaches U5.46 (PH5)
- net ph5: now also J5.4 (SDK), R20.1
- net gpio_stm32: now reaches U5.53 (PA7)
- net pb10: now reaches U5.79 (PB10)
- net pb10: now also J5.3 (SCK), R21.1
Other:
- moved on the sheet: J2
