File: electronics/lcd-unit-STM32/hs/lcd_con/lcd_con.kicad_sch (KiCad schematic)
At the start: 6 parts, among them J4 Conn_01x40

Commit message: Ambiente lighting draft, song order fixet for music rounds, many others
Parts:
- added C45: 4U7, Capacitor_SMD:C_0603_1608Metric, symbol Device:C_Small
- added C46: 100n, Capacitor_SMD:C_0603_1608Metric, symbol Device:C_Small
- added C47: 2.2u 50v, Capacitor_SMD:C_0603_1608Metric, symbol Device:C_Small
- added D7: D_Schottky, Diode_SMD:D_SMA, symbol Device:D_Schottky
- added L1: L, Inductor_SMD:L_Bourns-SRN4018, symbol Device:L
- added R11: 10R, Resistor_SMD:R_0805_2012Metric, symbol Device:R_Small
- added R16: 100R, Resistor_SMD:R_0805_2012Metric, symbol Device:R_Small
- added R17: 100K, Resistor_SMD:R_0805_2012Metric, symbol Device:R_Small
- added U6: TPS61169DCKR, moja:SOT65P210X110-5N, symbol moja:TPS61169DCKR
Connections:
- net +3V3: now also C45.1, C46.2, L1.2, U6.5 (VIN)
- net GND: now also C45.2, C46.1, C47.1, R11.1, R17.1, U6.2 (GND)
- net at J4.1 (ledk): now also R11.2, U6.3 (FB)
- net at J4.2 (led_a): now also C47.2, D7.1 (K)
- new net: D7.2 (A), L1.1, U6.1 (SW)
- new net: R16.2, U6.4 (CTRL)
- new net gpio_stm32: R16.1, R17.2
