File: electronics/main-unit/rayman_main.kicad_pcb (KiCad board)
At the start: 2 copper layers, 88 x 100 mm, 116 parts, among them M1 M1, M2 M2, Q1 BC817, T1A_FUSE1 1808 SMD FUSEHOLDER, U1 ESP32-S3-WROOM-1, U2 SN74AHCT125N, U3 SSR-DA41F, U4 MCP1826S-3302E/DB

Commit message: uv control fixed
Parts:
- removed R19: 100k, Resistor_SMD:R_0805_2012Metric
- added U5: SP3012-06UTG, moja:SON50P350X135X55-14N, F.Cu at (106.1, 45.8)
- R33: moved to F.Cu
- moved R33 35.9 mm to (96.4, 72.6)
- moved R22 0.65 mm to (107.1, 48.7)
- moved R27 0.65 mm to (111.5, 48.7)
- moved R25 0.65 mm to (109.3, 48.7)
- moved C12 0.65 mm to (102.6, 48.6)
- moved C13 0.65 mm to (104.8, 48.6)
Connections:
- R33 pad 2: io2 -> Net-(U2-4Y)
- U2 pad 11: unconnected-(U2-4Y-Pad11) -> Net-(U2-4Y)
- U2 pad 12: Net-(U2-4A) -> io2
Routing:
- net io2: track 24.6 -> 102.8 mm, vias 2 -> 3
- net Net-(R33-Pad1): track 128.2 -> 57.7 mm, vias 1 -> 2
- net Net-(U2-4Y): track 0.00 -> 21.4 mm
- net sd_miso: track 58.7 -> 37.6 mm, vias 0 -> 2
- net Net-(U2-4A): track 13.6 -> 0.00 mm, vias 1 -> 0
- net sd_cs: track 7.52 -> 13.7 mm, vias 0 -> 2
- net sd_mosi: track 14.4 -> 17.3 mm
- net sd_sck: track 28.0 -> 30.9 mm
- net GND: track 63.8 -> 65.7 mm, vias 29 -> 30
- net Net-(D10-A): track 116.5 -> 118.3 mm
- net Net-(TB1-PWMA): track 100.0 -> 101.5 mm
- net Net-(TB1-PWMB): track 110.0 -> 111.5 mm
- net +3V3: track 308.0 -> 306.6 mm, vias 9 -> 8
- net busy: track 36.4 -> 35.2 mm
- net Net-(U1-IO4): track 50.2 -> 49.3 mm
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
Commit message: Ambiente lighting draft, song order fixet for music rounds, many others
Parts:
- added C25: 100n, Capacitor_SMD:C_0805_2012Metric, F.Cu at (135.6, 114.5)
- added U6: STEF4SPUR, moja:STEF05PUR, F.Cu at (140.3, 114.4)
- R10, R11, R16, R17: value 10k -> 2k2
- R12: value 10k -> 100k
- R20, R21: value 2k2 -> 68R
- moved R14 65.9 mm to (144.7, 114.1)
- moved R12 8.17 mm to (81.1, 79.2), turned to 180 degrees
Connections:
- 1,0A_FUSE1 pad 2: +5V -> 5v_b4_prot
- 5VDC1 pad 2: +5V -> 5v_b4_prot
- R10 pad 2: Net-(R10-Pad2) -> Net-(C8-Pad1)
- R11 pad 2: Net-(R10-Pad2) -> Net-(C8-Pad1)
- R12 pad 1: Net-(C8-Pad1) -> Net-(audio_out1-DO)
- R12 pad 2: Net-(R10-Pad2) -> GND
- R14 pad 1: Net-(R14-Pad1) -> 5v_b4_prot
- R14 pad 2: Net-(C8-Pad1) -> Net-(U6-EN)
- R16 pad 2: Net-(R14-Pad1) -> Net-(C8-Pad1)
- R17 pad 2: Net-(R14-Pad1) -> Net-(C8-Pad1)
- R26 pad 1: Net-(D11-A) -> +5V
- TF1 pad G1: unconnected-(TF1-PadG1) -> GND
- TF1 pad G2: unconnected-(TF1-PadG2) -> GND
- TF1 pad G3: unconnected-(TF1-PadG3) -> GND
- TF1 pad G4: unconnected-(TF1-PadG4) -> GND
- U3 pad 3: Net-(D11-A) -> +5V
- U4 pad 1: Net-(D11-A) -> +5V
Routing:
- net Net-(D11-A): track 84.3 -> 43.3 mm, vias 3 -> 2
- net +5V: track 179.7 -> 217.0 mm, vias 2 -> 5
- net 5v_b4_prot: track 0.00 -> 33.1 mm
- net Net-(C8-Pad1): track 4.66 -> 15.1 mm
- net Net-(U6-EN): track 0.00 -> 8.85 mm
- net Net-(U6-SST): track 0.00 -> 8.62 mm, vias 0 -> 2
- net Net-(R14-Pad1): track 8.14 -> 0.00 mm
- net Net-(R10-Pad2): track 7.76 -> 0.00 mm
- net GND: track 65.7 -> 61.1 mm, vias 30 -> 31
- net Net-(audio_out1-DO): track 14.7 -> 19.2 mm
- net +3V3: track 306.6 -> 307.3 mm
- net Net-(FAN_L1-Pin_1): track 64.9 -> 64.2 mm
- net Net-(D5-A): track 4.43 -> 3.81 mm
- net Net-(D10-A): track 118.3 -> 118.8 mm
Other:
- board text added: "Rev 1.51 25-MAR-2026"
- board text removed: "Rev 1.5 25-MAR-2026"
